Commit message: Add fisheye camera

File: husky_description/urdf/husky.urdf.xacro (robot description, xacro)
@@ -145,5 +145,5 @@
         <plugin name="imu_controller" filename="libhector_gazebo_ros_imu.so">
             <robotNamespace>$(arg robot_namespace)</robotNamespace>
-            <updateRate>50.0</updateRate>
+            <updateRate>500.0</updateRate>
             <bodyName>base_link</bodyName>
             <topicName>imu/data</topicName>
@@ -171,5 +171,5 @@
     <!--  Left front camera  -->
     <joint name="left_camera_joint" type="fixed">
-        <origin xyz="${base_x_size/4} ${base_y_size/4} 0.1" />
+        <origin xyz="${base_x_size/4} ${base_y_size/4} 0.1"/>
         <parent link="top_plate_link"/>
         <child link="left_camera_frame"/>
@@ -188,14 +188,14 @@
     </link>
     <joint name="left_camera_optical_joint" type="fixed">
-        <origin xyz="0 0 0" rpy="${-M_PI/2} 0 ${-M_PI/2}" />
-        <parent link="left_camera_frame" />
-        <child link="left_camera_optical_frame" />
+        <origin xyz="0 0 0" rpy="${-M_PI/2} 0 ${-M_PI/2}"/>
+        <parent link="left_camera_frame"/>
+        <child link="left_camera_optical_frame"/>
     </joint>
     <link name="left_camera_optical_frame"/>
     <!-- Right front camera -->
     <joint name="right_camera_joint" type="fixed">
-        <origin xyz="${base_x_size/4} -${base_y_size/4} 0.1" />
+        <origin xyz="${base_x_size/4} -${base_y_size/4} 0.1"/>
         <parent link="top_plate_link"/>
-        <child link="right_camera_frame" />
+        <child link="right_camera_frame"/>
     </joint>
     <link name="right_camera_frame">
@@ -212,7 +212,7 @@
     </link>
     <joint name="right_camera_optical_joint" type="fixed">
-        <origin xyz="0 0 0" rpy="${-M_PI/2} 0 ${-M_PI/2}" />
-        <parent link="right_camera_frame" />
-        <child link="right_camera_optical_frame" />
+        <origin xyz="0 0 0" rpy="${-M_PI/2} 0 ${-M_PI/2}"/>
+        <parent link="right_camera_frame"/>
+        <child link="right_camera_optical_frame"/>
     </joint>
     <link name="right_camera_optical_frame"/>
@@ -221,5 +221,5 @@
         <origin xyz="-${base_x_size/4} 0 0.1" rpy="0 0 ${pi}"/>
         <parent link="top_plate_link"/>
-        <child link="rear_camera_frame" />
+        <child link="rear_camera_frame"/>
     </joint>
     <link name="rear_camera_frame">
@@ -236,9 +236,83 @@
     </link>
     <joint name="rear_camera_optical_joint" type="fixed">
-        <origin xyz="0 0 0" rpy="${-M_PI/2} 0 ${-M_PI/2}" />
-        <parent link="rear_camera_frame" />
-        <child link="rear_camera_optical_frame" />
+        <origin xyz="0 0 0" rpy="${-M_PI/2} 0 ${-M_PI/2}"/>
+        <parent link="rear_camera_frame"/>
+        <child link="rear_camera_optical_frame"/>
     </joint>
     <link name="rear_camera_optical_frame"/>
+    <!--
+    <gazebo reference="rear_camera_frame">
+        <sensor name='rear_sensor' type='camera'>
+            <update_rate>30</update_rate>
+            <camera name="left_camera">
+                <horizontal_fov>${radians(90)}</horizontal_fov>
+                <image>
+                    <width>320</width>
+                    <height>240</height>
+                    <format>B8G8R8</format>
+                </image>
+                <clip>
+                    <near>0.01</near>
+                    <far>300</far>
+                </clip>
+                <noise>
+                    <type>gaussian</type>
+                    <mean>0.0</mean>
+                    <stddev>0.0005</stddev>
+                </noise>
+            </camera>
+            <plugin name="rear_camera_controller" filename="libgazebo_ros_camera.so">
+                <alwaysOn>true</alwaysOn>
+                <updateRate>0</updateRate>
+                <cameraName>camera/left</cameraName>
+                <imageTopicName>image_raw</imageTopicName>
+                <cameraInfoTopicName>camera_info</cameraInfoTopicName>
+                <frameName>left_camera_optical_frame</frameName>
+                <distortionK1>0.0</distortionK1>
+                <distortionK2>0.0</distortionK2>
+                <distortionK3>0.0</distortionK3>
+                <distortionT1>0.0</distortionT1>
+                <distortionT2>0.0</distortionT2>
+            </plugin>
+        </sensor>
+    </gazebo>
+    -->
+    <gazebo reference="left_camera_frame">
+        <sensor name="left_camera" type="wideanglecamera">
+            <update_rate>25</update_rate>
+            <always_on>true</always_on>
+            <camera>
+                <!-- 185 degrees -->
+                <horizontal_fov>${radians(185)}</horizontal_fov>
+                <image>
+                    <width>754</width>
+                    <height>480</height>
+                </image>
+                <clip>
+                    <near>0.1</near>
+                    <far>100</far>
+                </clip>
+                <lens>
+                    <type>orthographic</type>
+                    <!-- if it is set to `true` your horizontal FOV will remain as defined -->
+                    <!-- otherwise it depends on lens type and custom function, if there is one -->
+                    <scale_to_hfov>false</scale_to_hfov>
+                    <!-- clip everything that is outside of this angle -->
+                    <!--<cutoff_angle>${pi/2]</cutoff_angle>-->
+                    <!-- resolution of the cube-map texture, the higher it is - the sharper is your image -->
+                    <env_texture_size>2048</env_texture_size>
+                </lens>
+            </camera>
+            <plugin name="camera_controller" filename="libgazebo_ros_camera.so">
+                <alwaysOn>true</alwaysOn>
+                <updateRate>0</updateRate>
+                <cameraName>camera/left</cameraName>
+                <imageTopicName>image_raw</imageTopicName>
+                <cameraInfoTopicName>camera_info</cameraInfoTopicName>
+                <frameName>left_camera_optical_frame</frameName>
+                <hackBaseline>0.0</hackBaseline>
+            </plugin>
+        </sensor>
+    </gazebo>
     <!-- Optional custom includes. -->
     <xacro:include filename="$(arg urdf_extras)"/>

Commit message: Fix

File: husky_description/urdf/husky.urdf.xacro (robot description, xacro)
@@ -188,5 +188,5 @@
     </link>
     <joint name="left_camera_optical_joint" type="fixed">
-        <origin xyz="0 0 0" rpy="${-M_PI/2} 0 ${-M_PI/2}"/>
+        <origin xyz="0 0 0" rpy="${-pi/2} 0 ${-pi/2}"/>
         <parent link="left_camera_frame"/>
         <child link="left_camera_optical_frame"/>
@@ -212,5 +212,5 @@
     </link>
     <joint name="right_camera_optical_joint" type="fixed">
-        <origin xyz="0 0 0" rpy="${-M_PI/2} 0 ${-M_PI/2}"/>
+        <origin xyz="0 0 0" rpy="${-pi/2} 0 ${-pi/2}"/>
         <parent link="right_camera_frame"/>
         <child link="right_camera_optical_frame"/>
@@ -236,5 +236,5 @@
     </link>
     <joint name="rear_camera_optical_joint" type="fixed">
-        <origin xyz="0 0 0" rpy="${-M_PI/2} 0 ${-M_PI/2}"/>
+        <origin xyz="0 0 0" rpy="${-pi/2} 0 ${-pi/2}"/>
         <parent link="rear_camera_frame"/>
         <child link="rear_camera_optical_frame"/>
@@ -254,5 +254,5 @@
                 </image>
                 <clip>
-                    <near>0.1</near>
+                    <near>0.02</near>
                     <far>100</far>
                 </clip>
@@ -265,5 +265,5 @@
                     <!--<cutoff_angle>${pi/2]</cutoff_angle>-->
                     <!-- resolution of the cube-map texture, the higher it is - the sharper is your image -->
-                    <env_texture_size>2048</env_texture_size>
+                    <env_texture_size>1024</env_texture_size>
                 </lens>
             </camera>
@@ -289,5 +289,5 @@
                 </image>
                 <clip>
-                    <near>0.1</near>
+                    <near>0.02</near>
                     <far>100</far>
                 </clip>
@@ -295,6 +295,5 @@
                     <type>orthographic</type>
                     <scale_to_hfov>false</scale_to_hfov>
-                    <!--<cutoff_angle>${pi/2]</cutoff_angle>-->
-                    <env_texture_size>2048</env_texture_size>
+                    <env_texture_size>1024</env_texture_size>
                 </lens>
             </camera>
@@ -320,5 +319,5 @@
                 </image>
                 <clip>
-                    <near>0.1</near>
+                    <near>0.02</near>
                     <far>100</far>
                 </clip>
@@ -326,6 +325,5 @@
                     <type>orthographic</type>
                     <scale_to_hfov>false</scale_to_hfov>
-                    <!--<cutoff_angle>${pi/2]</cutoff_angle>-->
-                    <env_texture_size>2048</env_texture_size>
+                    <env_texture_size>1024</env_texture_size>
                 </lens>
             </camera>

Commit message: Fix

File: husky_description/urdf/husky.urdf.xacro (robot description, xacro)
@@ -171,5 +171,5 @@
     <!--  Left front camera  -->
     <joint name="left_camera_joint" type="fixed">
-        <origin xyz="${base_x_size/4} ${base_y_size/4} 0.1"/>
+        <origin xyz="${base_x_size/4} ${base_y_size/4} 0.1" rpy="0 0 0"/>
         <parent link="top_plate_link"/>
         <child link="left_camera_frame"/>
@@ -195,5 +195,5 @@
     <!-- Right front camera -->
     <joint name="right_camera_joint" type="fixed">
-        <origin xyz="${base_x_size/4} -${base_y_size/4} 0.1"/>
+        <origin xyz="${base_x_size/4} -${base_y_size/4} 0.1" rpy="0 0 ${-pi/6}"/>
         <parent link="top_plate_link"/>
         <child link="right_camera_frame"/>
@@ -219,5 +219,5 @@
     <!-- Rear central camera -->
     <joint name="rear_camera_joint" type="fixed">
-        <origin xyz="-${base_x_size/4} 0 0.1" rpy="0 0 ${pi}"/>
+        <origin xyz="-${base_x_size/4} 0 0.1" rpy="0 0 ${2*pi/3}"/>
         <parent link="top_plate_link"/>
         <child link="rear_camera_frame"/>

Commit message: Pheonix

File: husky_description/urdf/husky.urdf.xacro (robot description, xacro)
@@ -171,5 +171,5 @@
     <!--  Left front camera  -->
     <joint name="left_camera_joint" type="fixed">
-        <origin xyz="${base_x_size/4} ${base_y_size/4} 0.1" rpy="0 0 0"/>
+        <origin xyz="0.1 0.1 0.5" rpy="0 0 0"/>
         <parent link="top_plate_link"/>
         <child link="left_camera_frame"/>
@@ -178,5 +178,5 @@
         <visual>
             <geometry>
-                <box size="0.1 0.1 0.2"/>
+                <box size="0.02 0.02 0.05"/>
             </geometry>
         </visual>
@@ -195,5 +195,5 @@
     <!-- Right front camera -->
     <joint name="right_camera_joint" type="fixed">
-        <origin xyz="${base_x_size/4} -${base_y_size/4} 0.1" rpy="0 0 ${-pi/6}"/>
+        <origin xyz="0.05 -0.1 0.5" rpy="0 0 ${-pi/3}"/>
         <parent link="top_plate_link"/>
         <child link="right_camera_frame"/>
@@ -202,5 +202,5 @@
         <visual>
             <geometry>
-                <box size="0.1 0.1 0.2"/>
+                <box size="0.02 0.02 0.05"/>
             </geometry>
         </visual>
@@ -219,5 +219,5 @@
     <!-- Rear central camera -->
     <joint name="rear_camera_joint" type="fixed">
-        <origin xyz="-${base_x_size/4} 0 0.1" rpy="0 0 ${2*pi/3}"/>
+        <origin xyz="-0.2 0 0.5" rpy="0 0 ${2*pi/3}"/>
         <parent link="top_plate_link"/>
         <child link="rear_camera_frame"/>
@@ -226,5 +226,5 @@
         <visual>
             <geometry>
-                <box size="0.1 0.1 0.2"/>
+                <box size="0.02 0.02 0.05"/>
             </geometry>
         </visual>
@@ -243,10 +243,9 @@
     <!-- Gazebo camera plugins -->
     <gazebo reference="left_camera_frame">
-        <sensor name="left_camera" type="camera">
+        <sensor name="left_camera" type="wideanglecamera">
             <update_rate>25</update_rate>
             <always_on>true</always_on>
             <camera>
-                <!-- 185 degrees -->
-                <horizontal_fov>${radians(89)}</horizontal_fov>
+                <horizontal_fov>${radians(185)}</horizontal_fov>
                 <image>
                     <width>754</width>
@@ -257,4 +256,10 @@
                     <far>100</far>
                 </clip>
+                <lense>
+                    <type>orthographic</type>
+                    <scale_to_hfov>true</scale_to_hfov>
+                    <cutoff_angle>${pi/2}</cutoff_angle>
+                    <env_texture_size>1024</env_texture_size>
+                </lense>
             </camera>
             <plugin name="left_camera_controller" filename="libgazebo_ros_camera.so">
@@ -269,9 +274,9 @@
     </gazebo>
     <gazebo reference="right_camera_frame">
-        <sensor name="right_camera" type="camera">
+        <sensor name="right_camera" type="wideanglecamera">
             <update_rate>25</update_rate>
             <always_on>true</always_on>
             <camera>
-                <horizontal_fov>${radians(89)}</horizontal_fov>
+                <horizontal_fov>${radians(185)}</horizontal_fov>
                 <image>
                     <width>754</width>
@@ -282,4 +287,10 @@
                     <far>100</far>
                 </clip>
+                <lense>
+                    <type>orthographic</type>
+                    <scale_to_hfov>true</scale_to_hfov>
+                    <cutoff_angle>${pi/2}</cutoff_angle>
+                    <env_texture_size>1024</env_texture_size>
+                </lense>
             </camera>
             <plugin name="right_camera_controller" filename="libgazebo_ros_camera.so">
@@ -294,9 +305,9 @@
     </gazebo>
     <gazebo reference="rear_camera_frame">
-        <sensor name="rear_camera" type="camera">
+        <sensor name="rear_camera" type="wideanglecamera">
             <update_rate>25</update_rate>
             <always_on>true</always_on>
             <camera>
-                <horizontal_fov>${radians(89)}</horizontal_fov>
+                <horizontal_fov>${radians(185)}</horizontal_fov>
                 <image>
                     <width>754</width>
@@ -307,4 +318,10 @@
                     <far>100</far>
                 </clip>
+                <lense>
+                    <type>orthographic</type>
+                    <scale_to_hfov>true</scale_to_hfov>
+                    <cutoff_angle>${pi/2}</cutoff_angle>
+                    <env_texture_size>1024</env_texture_size>
+                </lense>
             </camera>
             <plugin name="rear_camera_controller" filename="libgazebo_ros_camera.so">

Commit message: Move cameras. Custom config

File: husky_description/urdf/husky.urdf.xacro (robot description, xacro)
@@ -171,5 +171,5 @@
     <!--  Left front camera  -->
     <joint name="left_camera_joint" type="fixed">
-        <origin xyz="0.1 0.1 0.5" rpy="0 0 0"/>
+        <origin xyz="0.3 0.3 0.5" rpy="0 0 0"/>
         <parent link="top_plate_link"/>
         <child link="left_camera_frame"/>
@@ -195,5 +195,5 @@
     <!-- Right front camera -->
     <joint name="right_camera_joint" type="fixed">
-        <origin xyz="0.05 -0.1 0.5" rpy="0 0 ${-pi/3}"/>
+        <origin xyz="0.05 -0.3 0.5" rpy="0 0 ${-pi/3}"/>
         <parent link="top_plate_link"/>
         <child link="right_camera_frame"/>
@@ -219,5 +219,5 @@
     <!-- Rear central camera -->
     <joint name="rear_camera_joint" type="fixed">
-        <origin xyz="-0.2 0 0.5" rpy="0 0 ${2*pi/3}"/>
+        <origin xyz="-0.5 0 0.5" rpy="0 0 ${2*pi/3}"/>
         <parent link="top_plate_link"/>
         <child link="rear_camera_frame"/>
@@ -242,4 +242,27 @@
     <link name="rear_camera_optical_frame"/>
     <!-- Gazebo camera plugins -->
+    <xacro:macro name="camera_params">
+        <horizontal_fov>${radians(185)}</horizontal_fov>
+        <image>
+            <width>754</width>
+            <height>480</height>
+        </image>
+        <clip>
+            <near>0.15</near>
+            <far>100</far>
+        </clip>
+        <lense>
+            <type>custom</type>
+            <custom_function>
+                <c1>2</c1>
+                <c2>1</c2>
+                <f>1.25</f>
+                <fun>sin</fun>
+            </custom_function>
+            <scale_to_hfov>true</scale_to_hfov>
+            <cutoff_angle>${radians(185)}</cutoff_angle>
+            <env_texture_size>512</env_texture_size>
+        </lense>
+    </xacro:macro>
     <gazebo reference="left_camera_frame">
         <sensor name="left_camera" type="wideanglecamera">
@@ -247,19 +270,5 @@
             <always_on>true</always_on>
             <camera>
-                <horizontal_fov>${radians(185)}</horizontal_fov>
-                <image>
-                    <width>754</width>
-                    <height>480</height>
-                </image>
-                <clip>
-                    <near>0.02</near>
-                    <far>100</far>
-                </clip>
-                <lense>
-                    <type>orthographic</type>
-                    <scale_to_hfov>true</scale_to_hfov>
-                    <cutoff_angle>${pi/2}</cutoff_angle>
-                    <env_texture_size>1024</env_texture_size>
-                </lense>
+                <xacro:camera_params/>
             </camera>
             <plugin name="left_camera_controller" filename="libgazebo_ros_camera.so">
@@ -278,19 +287,5 @@
             <always_on>true</always_on>
             <camera>
-                <horizontal_fov>${radians(185)}</horizontal_fov>
-                <image>
-                    <width>754</width>
-                    <height>480</height>
-                </image>
-                <clip>
-                    <near>0.02</near>
-                    <far>100</far>
-                </clip>
-                <lense>
-                    <type>orthographic</type>
-                    <scale_to_hfov>true</scale_to_hfov>
-                    <cutoff_angle>${pi/2}</cutoff_angle>
-                    <env_texture_size>1024</env_texture_size>
-                </lense>
+                <xacro:camera_params/>
             </camera>
             <plugin name="right_camera_controller" filename="libgazebo_ros_camera.so">
@@ -309,19 +304,5 @@
             <always_on>true</always_on>
             <camera>
-                <horizontal_fov>${radians(185)}</horizontal_fov>
-                <image>
-                    <width>754</width>
-                    <height>480</height>
-                </image>
-                <clip>
-                    <near>0.02</near>
-                    <far>100</far>
-                </clip>
-                <lense>
-                    <type>orthographic</type>
-                    <scale_to_hfov>true</scale_to_hfov>
-                    <cutoff_angle>${pi/2}</cutoff_angle>
-                    <env_texture_size>1024</env_texture_size>
-                </lense>
+                <xacro:camera_params/>
             </camera>
             <plugin name="rear_camera_controller" filename="libgazebo_ros_camera.so">

Commit message: camera params

File: husky_description/urdf/husky.urdf.xacro (robot description, xacro)
@@ -178,5 +178,5 @@
         <visual>
             <geometry>
-                <box size="0.02 0.02 0.05"/>
+                <box size="0.0001 0.0001 0.0001"/>
             </geometry>
         </visual>
@@ -195,5 +195,5 @@
     <!-- Right front camera -->
     <joint name="right_camera_joint" type="fixed">
-        <origin xyz="0.05 -0.3 0.5" rpy="0 0 ${-pi/3}"/>
+        <origin xyz="0.05 -0.3 0.5" rpy="0 0 0"/>
         <parent link="top_plate_link"/>
         <child link="right_camera_frame"/>
@@ -202,5 +202,5 @@
         <visual>
             <geometry>
-                <box size="0.02 0.02 0.05"/>
+                <box size="0.0001 0.0001 0.0001"/>
             </geometry>
         </visual>
@@ -226,5 +226,5 @@
         <visual>
             <geometry>
-                <box size="0.02 0.02 0.05"/>
+                <box size="0.0001 0.0001 0.0001"/>
             </geometry>
         </visual>
@@ -255,12 +255,12 @@
             <type>custom</type>
             <custom_function>
-                <c1>2</c1>
-                <c2>1</c2>
-                <f>1.25</f>
+                <c1>1.0</c1>
+                <c2>1.5</c2>
+                <f>1.0</f>
                 <fun>sin</fun>
             </custom_function>
-            <scale_to_hfov>true</scale_to_hfov>
-            <cutoff_angle>${radians(185)}</cutoff_angle>
-            <env_texture_size>512</env_texture_size>
+<!--            <scale_to_hfov>true</scale_to_hfov>-->
+<!--            <cutoff_angle>${radians(90)}</cutoff_angle>-->
+            <env_texture_size>1024</env_texture_size>
         </lense>
     </xacro:macro>
