Commit message: Update description

File: husky_description/urdf/husky.urdf.xacro (robot description, xacro)
@@ -7,10 +7,10 @@
 Redistribution and use in source and binary forms, with or without modification, are permitted provided that
 the following conditions are met:
- * Redistributions of source code must retain the above copyright notice, this list of conditions and the
-   following disclaimer.
- * Redistributions in binary form must reproduce the above copyright notice, this list of conditions and the
-   following disclaimer in the documentation and/or other materials provided with the distribution.
- * Neither the name of Clearpath Robotics nor the names of its contributors may be used to endorse or promote
-   products derived from this software without specific prior written permission.
+* Redistributions of source code must retain the above copyright notice, this list of conditions and the
+ following disclaimer.
+* Redistributions in binary form must reproduce the above copyright notice, this list of conditions and the
+ following disclaimer in the documentation and/or other materials provided with the distribution.
+* Neither the name of Clearpath Robotics nor the names of its contributors may be used to endorse or promote
+ products derived from this software without specific prior written permission.
 THIS SOFTWARE IS PROVIDED BY THE COPYRIGHT HOLDERS AND CONTRIBUTORS "AS IS" AND ANY EXPRESS OR IMPLIED WAR-
 RANTIES, INCLUDING, BUT NOT LIMITED TO, THE IMPLIED WARRANTIES OF MERCHANTABILITY AND FITNESS FOR A PARTICULAR
@@ -22,323 +22,316 @@
 -->
 <robot name="husky" xmlns:xacro="http://ros.org/wiki/xacro">
-    <xacro:arg name="laser_enabled" default="false"/>
-    <xacro:arg name="laser_xyz" default="$(optenv HUSKY_LMS1XX_XYZ 0.2206 0.0 0.00635)"/>
-    <xacro:arg name="laser_rpy" default="$(optenv HUSKY_LMS1XX_RPY 0.0 0.0 0.0)"/>
-    <xacro:arg name="kinect_enabled" default="false"/>
-    <xacro:arg name="kinect_xyz" default="$(optenv HUSKY_KINECT_XYZ 0 0 0)"/>
-    <xacro:arg name="kinect_rpy" default="$(optenv HUSKY_KINECT_RPY 0 0.18 3.14)"/>
-    <xacro:property name="husky_front_bumper_extend" value="$(optenv HUSKY_FRONT_BUMPER_EXTEND 0)"/>
-    <xacro:property name="husky_rear_bumper_extend" value="$(optenv HUSKY_REAR_BUMPER_EXTEND 0)"/>
-    <xacro:arg name="robot_namespace" default="/"/>
-    <xacro:arg name="urdf_extras" default="empty.urdf"/>
-    <!-- Included URDF/XACRO Files -->
-    <xacro:include filename="$(find husky_description)/urdf/decorations.urdf.xacro"/>
-    <xacro:include filename="$(find husky_description)/urdf/wheel.urdf.xacro"/>
-    <xacro:include filename="$(find husky_description)/urdf/accessories/kinect_camera.urdf.xacro"/>
-    <xacro:include filename="$(find husky_description)/urdf/accessories/sick_lms1xx_mount.urdf.xacro"/>
-    <xacro:include filename="$(find husky_description)/urdf/accessories/sensor_arch.urdf.xacro"/>
-    <xacro:property name="M_PI" value="3.14159"/>
-    <!-- Base Size -->
-    <xacro:property name="base_x_size" value="0.98740000"/>
-    <xacro:property name="base_y_size" value="0.57090000"/>
-    <xacro:property name="base_z_size" value="0.24750000"/>
-    <!-- Wheel Mounting Positions -->
-    <xacro:property name="wheelbase" value="0.5120"/>
-    <xacro:property name="track" value="0.5708"/>
-    <xacro:property name="wheel_vertical_offset" value="0.03282"/>
-    <!-- Wheel Properties -->
-    <xacro:property name="wheel_length" value="0.1143"/>
-    <xacro:property name="wheel_radius" value="0.1651"/>
-    <!-- Base link is the center of the robot's bottom plate -->
-    <link name="base_link">
-        <visual>
-            <origin xyz="0 0 0" rpy="0 0 0"/>
-            <geometry>
-                <mesh filename="package://husky_description/meshes/base_link.dae"/>
-            </geometry>
-        </visual>
-        <collision>
-            <origin xyz="${( husky_front_bumper_extend - husky_rear_bumper_extend ) / 2.0} 0 ${base_z_size/4}"
-                    rpy="0 0 0"/>
-            <geometry>
-                <box size="${ base_x_size + husky_front_bumper_extend + husky_rear_bumper_extend } ${base_y_size} ${base_z_size/2}"/>
-            </geometry>
-        </collision>
-        <collision>
-            <origin xyz="0 0 ${base_z_size*3/4-0.01}" rpy="0 0 0"/>
-            <geometry>
-                <box size="${base_x_size*4/5} ${base_y_size} ${base_z_size/2-0.02}"/>
-            </geometry>
-        </collision>
-    </link>
-    <!-- Base footprint is on the ground under the robot -->
-    <link name="base_footprint"/>
-    <joint name="base_footprint_joint" type="fixed">
-        <origin xyz="0 0 ${wheel_vertical_offset - wheel_radius}" rpy="0 0 0"/>
-        <parent link="base_link"/>
-        <child link="base_footprint"/>
+  <xacro:arg name="laser_enabled" default="false"/>
+  <xacro:arg name="laser_xyz" default="$(optenv HUSKY_LMS1XX_XYZ 0.2206 0.0 0.00635)"/>
+  <xacro:arg name="laser_rpy" default="$(optenv HUSKY_LMS1XX_RPY 0.0 0.0 0.0)"/>
+  <xacro:arg name="kinect_enabled" default="false"/>
+  <xacro:arg name="kinect_xyz" default="$(optenv HUSKY_KINECT_XYZ 0 0 0)"/>
+  <xacro:arg name="kinect_rpy" default="$(optenv HUSKY_KINECT_RPY 0 0.18 3.14)"/>
+  <xacro:property name="husky_front_bumper_extend" value="$(optenv HUSKY_FRONT_BUMPER_EXTEND 0)"/>
+  <xacro:property name="husky_rear_bumper_extend" value="$(optenv HUSKY_REAR_BUMPER_EXTEND 0)"/>
+  <xacro:arg name="robot_namespace" default="/"/>
+  <!-- Included URDF/XACRO Files -->
+  <xacro:include filename="$(find husky_description)/urdf/decorations.urdf.xacro"/>
+  <xacro:include filename="$(find husky_description)/urdf/wheel.urdf.xacro"/>
+  <xacro:include filename="$(find husky_description)/urdf/accessories/kinect_camera.urdf.xacro"/>
+  <xacro:include filename="$(find husky_description)/urdf/accessories/sick_lms1xx_mount.urdf.xacro"/>
+  <xacro:include filename="$(find husky_description)/urdf/accessories/sensor_arch.urdf.xacro"/>
+  <xacro:property name="M_PI" value="3.14159"/>
+  <!-- Base Size -->
+  <xacro:property name="base_x_size" value="0.98740000"/>
+  <xacro:property name="base_y_size" value="0.57090000"/>
+  <xacro:property name="base_z_size" value="0.24750000"/>
+  <!-- Wheel Mounting Positions -->
+  <xacro:property name="wheelbase" value="0.5120"/>
+  <xacro:property name="track" value="0.5708"/>
+  <xacro:property name="wheel_vertical_offset" value="0.03282"/>
+  <!-- Wheel Properties -->
+  <xacro:property name="wheel_length" value="0.1143"/>
+  <xacro:property name="wheel_radius" value="0.1651"/>
+  <!-- Base link is the center of the robot's bottom plate -->
+  <link name="base_link">
+    <visual>
+      <geometry>
+        <mesh filename="package://husky_description/meshes/base_link.dae"/>
+      </geometry>
+    </visual>
+    <collision>
+        <origin xyz="${( husky_front_bumper_extend - husky_rear_bumper_extend ) / 2.0} 0 ${base_z_size/4}"/>
+        <geometry>
+          <box size="${ base_x_size + husky_front_bumper_extend + husky_rear_bumper_extend } ${base_y_size} ${base_z_size/2}"/>
+        </geometry>
+    </collision>
+    <collision>
+        <origin xyz="0 0 ${base_z_size*3/4-0.01}" rpy="0 0 0"/>
+        <geometry>
+          <box size="${base_x_size*4/5} ${base_y_size} ${base_z_size/2-0.02}"/>
+        </geometry>
+    </collision>
+  </link>
+  <!-- Base footprint is on the ground under the robot -->
+  <link name="base_footprint"/>
+  <joint name="base_footprint_joint" type="fixed">
+    <origin xyz="0 0 ${wheel_vertical_offset - wheel_radius}" rpy="0 0 0"/>
+    <parent link="base_link"/>
+    <child link="base_footprint"/>
+  </joint>
+  <!-- Interial link stores the robot's inertial information -->
+  <link name="inertial_link">
+    <inertial>
+      <mass value="46.034"/>
+      <origin xyz="-0.00065 -0.085 0.062"/>
+      <inertia ixx="0.6022" ixy="-0.02364" ixz="-0.1197" iyy="1.7386" iyz="-0.001544" izz="2.0296"/>
+    </inertial>
+  </link>
+  <joint name="inertial_joint" type="fixed">
+    <origin xyz="0 0 0" rpy="0 0 0"/>
+    <parent link="base_link"/>
+    <child link="inertial_link"/>
+  </joint>
+  <!-- IMU Link is the standard mounting position for the UM6 IMU.-->
+  <!-- Can be modified with environment variables in /etc/ros/setup.bash -->
+  <link name="imu_link"/>
+    <joint name="imu_joint" type="fixed">
+      <origin xyz="$(optenv HUSKY_IMU_XYZ 0.19 0 0.149)" rpy="$(optenv HUSKY_IMU_RPY 0 -${pi/2} ${pi})"/>
+      <parent link="base_link"/>
+      <child link="imu_link"/>
     </joint>
-    <!-- Interial link stores the robot's inertial information -->
-    <link name="inertial_link">
-        <inertial>
-            <mass value="46.034"/>
-            <origin xyz="-0.00065 -0.085 0.062"/>
-            <inertia ixx="0.6022" ixy="-0.02364" ixz="-0.1197" iyy="1.7386" iyz="-0.001544" izz="2.0296"/>
-        </inertial>
-    </link>
-    <joint name="inertial_joint" type="fixed">
-        <origin xyz="0 0 0" rpy="0 0 0"/>
-        <parent link="base_link"/>
-        <child link="inertial_link"/>
-    </joint>
-    <!-- IMU Link is the standard mounting position for the UM6 IMU.-->
-    <!-- Can be modified with environment variables in /etc/ros/setup.bash -->
-    <link name="imu_link"/>
-    <joint name="imu_joint" type="fixed">
-        <origin xyz="$(optenv HUSKY_IMU_XYZ 0.19 0 0.149)" rpy="$(optenv HUSKY_IMU_RPY 0 -1.5708 3.1416)"/>
-        <parent link="base_link"/>
-        <child link="imu_link"/>
-    </joint>
-    <gazebo reference="imu_link">
-    </gazebo>
-    <!-- Husky wheel macros -->
-    <xacro:husky_wheel wheel_prefix="front_left">
-        <origin xyz="${wheelbase/2} ${track/2} ${wheel_vertical_offset}" rpy="0 0 0"/>
-    </xacro:husky_wheel>
-    <xacro:husky_wheel wheel_prefix="front_right">
-        <origin xyz="${wheelbase/2} ${-track/2} ${wheel_vertical_offset}" rpy="0 0 0"/>
-    </xacro:husky_wheel>
-    <xacro:husky_wheel wheel_prefix="rear_left">
-        <origin xyz="${-wheelbase/2} ${track/2} ${wheel_vertical_offset}" rpy="0 0 0"/>
-    </xacro:husky_wheel>
-    <xacro:husky_wheel wheel_prefix="rear_right">
-        <origin xyz="${-wheelbase/2} ${-track/2} ${wheel_vertical_offset}" rpy="0 0 0"/>
-    </xacro:husky_wheel>
-    <xacro:husky_decorate/>
-    <xacro:if value="$(arg laser_enabled)">
-        <sick_lms1xx_mount prefix="base"/>
-        <sick_lms1xx frame="base_laser" topic="scan" robot_namespace="$(arg robot_namespace)"/>
-        <joint name="laser_mount_joint" type="fixed">
-            <origin xyz="$(arg laser_xyz)" rpy="$(arg laser_rpy)"/>
-            <parent link="top_plate_link"/>
-            <child link="base_laser_mount"/>
-        </joint>
-    </xacro:if>
-    <xacro:if value="$(arg kinect_enabled)">
-        <xacro:sensor_arch prefix="" parent="top_plate_link">
-            <origin xyz="-0.35 0 0.51" rpy="0 0 -3.14"/>
-        </xacro:sensor_arch>
-        <joint name="kinect_frame_joint" type="fixed">
-            <origin xyz="$(arg kinect_xyz)" rpy="$(arg kinect_rpy)"/>
-            <parent link="sensor_arch_mount_link"/>
-            <child link="camera_link"/>
-        </joint>
-        <xacro:kinect_camera prefix="camera" robot_namespace="$(arg robot_namespace)"/>
-    </xacro:if>
-    <gazebo>
-        <plugin name="gazebo_ros_control" filename="libgazebo_ros_control.so">
-            <robotNamespace>$(arg robot_namespace)</robotNamespace>
-            <legacyModeNS>true</legacyModeNS>
-        </plugin>
-    </gazebo>
-    <gazebo>
-        <plugin name="imu_controller" filename="libhector_gazebo_ros_imu.so">
-            <robotNamespace>$(arg robot_namespace)</robotNamespace>
-            <updateRate>500.0</updateRate>
-            <bodyName>base_link</bodyName>
-            <topicName>imu/data</topicName>
-            <accelDrift>0.005 0.005 0.005</accelDrift>
-            <accelGaussianNoise>0.005 0.005 0.005</accelGaussianNoise>
-            <rateDrift>0.005 0.005 0.005</rateDrift>
-            <rateGaussianNoise>0.005 0.005 0.005</rateGaussianNoise>
-            <headingDrift>0.005</headingDrift>
-            <headingGaussianNoise>0.005</headingGaussianNoise>
-        </plugin>
-    </gazebo>
-    <!-- Ground truth -->
-    <gazebo>
-        <plugin filename="libgazebo_ros_p3d.so" name="gazebo_ros_p3d">
-            <alwaysOn>true</alwaysOn>
-            <updateRate>500.0</updateRate>
-            <!-- world frame is provided by Gazebo, it is not present in /tf topic -->
-            <frameName>world</frameName>
-            <bodyName>base_link</bodyName>
-            <topicName>ground_truth</topicName>
-            <xyzOffsets>0 0 0</xyzOffsets>
-            <rpyOffsets>0 0 0</rpyOffsets>
-        </plugin>
-    </gazebo>
-    <!--  Left front camera  -->
-    <joint name="left_camera_joint" type="fixed">
-        <origin xyz="${base_x_size/4} ${base_y_size/4} 0.1"/>
-        <parent link="top_plate_link"/>
-        <child link="left_camera_frame"/>
-    </joint>
-    <link name="left_camera_frame">
-        <visual>
-            <geometry>
-                <box size="0.1 0.1 0.2"/>
-            </geometry>
-        </visual>
-        <collision>
-            <geometry>
-                <box size="0.001 0.001 0.001"/>
-            </geometry>
-        </collision>
-    </link>
-    <joint name="left_camera_optical_joint" type="fixed">
-        <origin xyz="0 0 0" rpy="${-pi/2} 0 ${-pi/2}"/>
-        <parent link="left_camera_frame"/>
-        <child link="left_camera_optical_frame"/>
-    </joint>
-    <link name="left_camera_optical_frame"/>
-    <!-- Right front camera -->
-    <joint name="right_camera_joint" type="fixed">
-        <origin xyz="${base_x_size/4} -${base_y_size/4} 0.1"/>
-        <parent link="top_plate_link"/>
-        <child link="right_camera_frame"/>
-    </joint>
-    <link name="right_camera_frame">
-        <visual>
-            <geometry>
-                <box size="0.1 0.1 0.2"/>
-            </geometry>
-        </visual>
-        <collision>
-            <geometry>
-                <box size="0.001 0.001 0.001"/>
-            </geometry>
-        </collision>
-    </link>
-    <joint name="right_camera_optical_joint" type="fixed">
-        <origin xyz="0 0 0" rpy="${-pi/2} 0 ${-pi/2}"/>
-        <parent link="right_camera_frame"/>
-        <child link="right_camera_optical_frame"/>
-    </joint>
-    <link name="right_camera_optical_frame"/>
-    <!-- Rear central camera -->
-    <joint name="rear_camera_joint" type="fixed">
-        <origin xyz="-${base_x_size/4} 0 0.1" rpy="0 0 ${pi}"/>
-        <parent link="top_plate_link"/>
-        <child link="rear_camera_frame"/>
-    </joint>
-    <link name="rear_camera_frame">
-        <visual>
-            <geometry>
-                <box size="0.1 0.1 0.2"/>
-            </geometry>
-        </visual>
-        <collision>
-            <geometry>
-                <box size="0.001 0.001 0.001"/>
-            </geometry>
-        </collision>
-    </link>
-    <joint name="rear_camera_optical_joint" type="fixed">
-        <origin xyz="0 0 0" rpy="${-pi/2} 0 ${-pi/2}"/>
-        <parent link="rear_camera_frame"/>
-        <child link="rear_camera_optical_frame"/>
-    </joint>
-    <link name="rear_camera_optical_frame"/>
-    <!-- Gazebo camera plugins -->
-    <gazebo reference="left_camera_frame">
-        <sensor name="left_camera" type="wideanglecamera">
-            <update_rate>25</update_rate>
-            <always_on>true</always_on>
-            <camera>
-                <!-- 185 degrees -->
-                <horizontal_fov>${radians(185)}</horizontal_fov>
-                <image>
-                    <width>754</width>
-                    <height>480</height>
-                </image>
-                <clip>
-                    <near>0.02</near>
-                    <far>100</far>
-                </clip>
-                <lens>
-                    <type>orthographic</type>
-                    <!-- if it is set to `true` your horizontal FOV will remain as defined -->
-                    <!-- otherwise it depends on lens type and custom function, if there is one -->
-                    <scale_to_hfov>true</scale_to_hfov>
-                    <!-- clip everything that is outside of this angle -->
-                    <cutoff_angle>${pi/2]</cutoff_angle>
-                    <!-- resolution of the cube-map texture, the higher it is - the sharper is your image -->
-                    <env_texture_size>512</env_texture_size>
-                </lens>
-            </camera>
-            <plugin name="left_camera_controller" filename="libgazebo_ros_camera.so">
-                <alwaysOn>true</alwaysOn>
-                <updateRate>0</updateRate>
-                <cameraName>camera/left</cameraName>
-                <imageTopicName>image_raw</imageTopicName>
-                <cameraInfoTopicName>camera_info</cameraInfoTopicName>
-                <frameName>left_camera_optical_frame</frameName>
-            </plugin>
-        </sensor>
-    </gazebo>
-    <gazebo reference="right_camera_frame">
-        <sensor name="right_camera" type="wideanglecamera">
-            <update_rate>25</update_rate>
-            <always_on>true</always_on>
-            <camera>
-                <horizontal_fov>${radians(185)}</horizontal_fov>
-                <image>
-                    <width>754</width>
-                    <height>480</height>
-                </image>
-                <clip>
-                    <near>0.02</near>
-                    <far>100</far>
-                </clip>
-                <lens>
-                    <type>orthographic</type>
-                    <scale_to_hfov>true</scale_to_hfov>
-                    <cutoff_angle>${pi/2]</cutoff_angle>
-                    <env_texture_size>512</env_texture_size>
-                </lens>
-            </camera>
-            <plugin name="right_camera_controller" filename="libgazebo_ros_camera.so">
-                <alwaysOn>true</alwaysOn>
-                <updateRate>0</updateRate>
-                <cameraName>camera/right</cameraName>
-                <imageTopicName>image_raw</imageTopicName>
-                <cameraInfoTopicName>camera_info</cameraInfoTopicName>
-                <frameName>right_camera_optical_frame</frameName>
-            </plugin>
-        </sensor>
-    </gazebo>
-    <gazebo reference="rear_camera_frame">
-        <sensor name="rear_camera" type="wideanglecamera">
-            <update_rate>25</update_rate>
-            <always_on>true</always_on>
-            <camera>
-                <horizontal_fov>${radians(185)}</horizontal_fov>
-                <image>
-                    <width>754</width>
-                    <height>480</height>
-                </image>
-                <clip>
-                    <near>0.02</near>
-                    <far>100</far>
-                </clip>
-                <lens>
-                    <type>orthographic</type>
-                    <scale_to_hfov>true</scale_to_hfov>
-                    <cutoff_angle>${pi/2]</cutoff_angle>
-                    <env_texture_size>512</env_texture_size>
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